Commit message: test first 3 joint and links

File: neobotix_schunk_pybullet/data/neobotixschunk/mp500lwa4d_test.urdf (robot description, URDF)
Before this commit: robot mp500lwa4d_robot, 20 links, 19 joints
Links:
- removed link arm_1_link
- removed link arm_2_link
- removed link arm_3_link
- removed link arm_4_link
- removed link arm_5_link
- removed link arm_6_link
- removed link arm_7_link
- removed link arm_base_link
- removed link arm_podest_link
- removed link grasping_frame
- removed link gripper_finger_left_link
- removed link gripper_finger_right_link
- removed link gripper_palm_link
- removed link gripper_podest_link
- removed link laserscanner_front_link
- link base_link: geometry collision mesh filename=package://neobotix_schunk_pybullet/data/neobotixschunk/mesh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 scale=0.01 0.01 0.01; visual mesh filename=package://neobotix_schunk_pybullet/data/neobotixschunk/mesh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 scale=0.01 0.01 0.01
- link hanger: geometry collision sphere radius=0.125; visual sphere radius=0.125
Joints:
- removed joint arm_1_joint
- removed joint arm_2_joint
- removed joint arm_3_joint
- removed joint arm_4_joint
- removed joint arm_5_joint
- removed joint arm_6_joint
- removed joint arm_7_joint
- removed joint arm_base_joint
- removed joint arm_podest_joint
- removed joint grasping_frame_joint
- removed joint gripper_finger_left_joint
- removed joint gripper_finger_right_joint
- removed joint gripper_palm_joint
- removed joint gripper_podest_joint
- removed joint laserscanner_front_joint
- joint hanger_joint: origin xyz=0.255 0 0.125 rpy=0 0 0 -> xyz=0.415 0 0.125 rpy=0 0 0
- joint wheel_left_joint: origin xyz=-0.155 0.255 0.125 rpy=0 0 0 -> xyz=-0.01 0.255 0.125 rpy=0 0 0
- joint wheel_right_joint: origin xyz=-0.155 -0.255 0.125 rpy=0 0 0 -> xyz=-0.01 -0.255 0.125 rpy=0 0 0

Commit message: fix the model, the fz of joint 5 and 6 are now normal

File: neobotix_schunk_pybullet/data/neobotixschunk/mp500lwa4d_test.urdf (robot description, URDF)
Before this commit: robot mp500lwa4d_robot, 5 links, 4 joints
Links:
- added link arm_1_link, mass 0.01; collision mesh filename=package://neobotix_schunk_pybullet/data/neobotixschunk/mesh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; visual mesh filename=package://neobotix_schunk_pybullet/data/neobotixschunk/mesh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
- added link arm_2_link, mass 0.01; collision mesh filename=package://neobotix_schunk_pybullet/data/neobotixschunk/mesh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; visual mesh filename=package://neobotix_schunk_pybullet/data/neobotixschunk/mesh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
- added link arm_3_link, mass 0.01; collision mesh filename=package://neobotix_schunk_pybullet/data/neobotixschunk/mesh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; visual mesh filename=package://neobotix_schunk_pybullet/data/neobotixschunk/mesh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
- added link arm_4_link, mass 0.01; collision mesh filename=package://neobotix_schunk_pybullet/data/neobotixschunk/mesh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; visual mesh filename=package://neobotix_schunk_pybullet/data/neobotixschunk/mesh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
- added link arm_5_link, mass 0.01; collision mesh filename=package://neobotix_schunk_pybullet/data/neobotixschunk/mesh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; visual mesh filename=package://neobotix_schunk_pybullet/data/neobotixschunk/mesh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
- added link arm_6_link, mass 0.01; collision mesh filename=package://neobotix_schunk_pybullet/data/neobotixschunk/mesh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 scale=0.9 0.9 0.9; visual mesh filename=package://neobotix_schunk_pybullet/data/neobotixschunk/mesh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
- added link arm_7_link, mass 0.01; collision mesh filename=package://neobotix_schunk_pybullet/data/neobotixschunk/mesh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 scale=0.9 0.9 0.9; visual mesh filename=package://neobotix_schunk_pybullet/data/neobotixschunk/mesh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
- added link arm_base_link, mass 0.01
- added link arm_podest_link, mass 0.01; collision mesh filename=package://neobotix_schunk_pybullet/data/neobotixschunk/mesh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; visual mesh filename=package://neobotix_schunk_pybullet/data/neobotixschunk/mesh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
- added link grasping_frame, mass 0.0001
- added link gripper_finger_left_link, mass 0.001; collision box size=0.03 0.005 0.08; visual box size=0.03 0.01 0.08
- added link gripper_finger_right_link, mass 0.001; collision box size=0.03 0.005 0.08; visual box size=0.03 0.01 0.08
- added link gripper_palm_link, mass 0.001; collision box size=0.082 0.114 0.080; visual mesh filename=package://neobotix_schunk_pybullet/data/neobotixschunk/mesh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
- added link gripper_podest_link, mass 0.01; collision mesh filename=package://neobotix_schunk_pybullet/data/neobotixschunk/mesh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; visual mesh filename=package://neobotix_schunk_pybullet/data/neobotixschunk/mesh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
- added link laserscanner_front_link, mass 0.01; collision cylinder length=0.154 radius=0.053; visual mesh filename=package://neobotix_schunk_pybullet/data/neobotixschunk/mesh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
Joints:
- added joint arm_1_joint: type revolute, parent arm_base_link, child arm_1_link, origin xyz=0 0 0.019 rpy=0 0 0, axis 0 0 1, limit lower=-3.12159265359 upper=3.12159265359 effort=216 velocity=0.43633
- added joint arm_2_joint: type revolute, parent arm_1_link, child arm_2_link, origin xyz=0 0 0.24 rpy=-1.57079632679 -1.57079632679 0, axis 0 0 1, limit lower=-2.12 upper=2.12 effort=216 velocity=0.43633
- added joint arm_3_joint: type revolute, parent arm_2_link, child arm_3_link, origin xyz=0 0 0 rpy=1.57079632679 0 1.57079632679, axis 0 0 1, limit lower=-3.12159265359 upper=3.12159265359 effort=81.5 velocity=0.4189
- added joint arm_4_joint: type revolute, parent arm_3_link, child arm_4_link, origin xyz=0 0 0.328 rpy=-1.57079632679 -1.57079632679 0, axis 0 0 1, limit lower=-2.16 upper=2.16 effort=81.5 velocity=0.4189
- added joint arm_5_joint: type revolute, parent arm_4_link, child arm_5_link, origin xyz=0 0 0 rpy=1.57079632679 0 1.57079632679, axis 0 0 1, limit lower=-3.12159265359 upper=3.12159265359 effort=20.7 velocity=0.43633
- added joint arm_6_joint: type revolute, parent arm_5_link, child arm_6_link, origin xyz=0.00 0.00 0.323 rpy=-1.57079632679 -1.57079632679 0, axis 0 0 1, limit lower=-2.94 upper=2.94 effort=15 velocity=1.2566
- added joint arm_7_joint: type revolute, parent arm_6_link, child arm_7_link, origin xyz=0.00 0 0 rpy=1.57079632679 0 1.57079632679, axis 0 0 1, limit lower=-2.94 upper=2.94 effort=15 velocity=1.2566
- added joint arm_base_joint: type fixed, parent arm_podest_link, child arm_base_link, origin xyz=0 0 0.141 rpy=0 0 0, axis 0 0 1
- added joint arm_podest_joint: type fixed, parent base_link, child arm_podest_link, origin xyz=0.35 0 0.36 rpy=0 0 0
- added joint grasping_frame_joint: type fixed, parent arm_7_link, child grasping_frame, origin xyz=0 0 0.2463 rpy=0 0 0
- added joint gripper_finger_left_joint: type fixed, parent gripper_palm_link, child gripper_finger_left_link, origin xyz=0 -0.025 0.1139 rpy=0 0 0, axis 0 1 0, limit lower=-0.0301 upper=-0.01 effort=10 velocity=0.041
- added joint gripper_finger_right_joint: type fixed, parent gripper_palm_link, child gripper_finger_right_link, origin xyz=0 0.025 0.1139 rpy=-0 0 0, axis 0 1 0, limit lower=0.01 upper=0.0301 effort=10 velocity=0.041
- added joint gripper_palm_joint: type fixed, parent gripper_podest_link, child gripper_palm_link, origin xyz=0 0 0 rpy=0 0 0
- added joint gripper_podest_joint: type fixed, parent arm_7_link, child gripper_podest_link, origin xyz=0 0 0.1324 rpy=0 0 0
- added joint laserscanner_front_joint: type fixed, parent base_link, child laserscanner_front_link, origin xyz=-0.23 0 0.281 rpy=0 0 0, axis 0 0 1

Commit message: have fixed the model

File: neobotix_schunk_pybullet/data/neobotixschunk/mp500lwa4d_test.urdf (robot description, URDF)
Before this commit: robot mp500lwa4d_robot, 20 links, 19 joints
Links:
- link arm_5_link: geometry collision mesh filename=package://neobotix_schunk_pybullet/data/neobotixschunk/mesh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 scale=0.8 0.8 0.8; visual mesh filename=package://neobotix_schunk_pybullet/data/neobotixschunk/mesh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
- link arm_6_link: geometry collision sphere radius=0.04; visual sphere radius=0.04
- link arm_7_link: geometry collision mesh filename=package://neobotix_schunk_pybullet/data/neobotixschunk/mesh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 scale=0.8 0.8 0.8; visual mesh filename=package://neobotix_schunk_pybullet/data/neobotixschunk/mesh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
- link hanger: geometry collision sphere radius=0.125; visual mesh filename=package://neobotix_schunk_pybullet/data/neobotixschunk/mesh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 scale=0.01 0.01 0.01
