Commit message: add praktikum recorder and pictures

File: neobotix_schunk_pybullet/data/neobotixschunk/mp500lwa4d_2.urdf (robot description, URDF)
Before this commit: robot mp500lwa4d_robot, 20 links, 19 joints
Links:
- link arm_1_link: geometry collision mesh filename=/data/neobotixschunk/meshes/arm_1_link.stl; visual mesh filename=/data/neobotixschunk/meshes/arm_1_link.stl
- link arm_2_link: geometry collision mesh filename=/data/neobotixschunk/meshes/arm_2_link_collision.stl; visual mesh filename=/data/neobotixschunk/meshes/arm_2_link.stl
- link arm_3_link: geometry collision mesh filename=/data/neobotixschunk/meshes/arm_3_link_collision.stl; visual mesh filename=/data/neobotixschunk/meshes/arm_3_link.stl
- link arm_4_link: geometry collision mesh filename=/data/neobotixschunk/meshes/arm_4_link_collision.stl; visual mesh filename=/data/neobotixschunk/meshes/arm_4_link.stl
- link arm_5_link: geometry collision mesh filename=/data/neobotixschunk/meshes/arm_5_link_collision.stl scale=0.8 0.8 0.8; visual mesh filename=/data/neobotixschunk/meshes/arm_5_link.stl
- link arm_6_link: geometry collision mesh filename=/data/neobotixschunk/meshes/arm_6_link_collision.stl scale=0.9 0.9 0.9; visual mesh filename=/data/neobotixschunk/meshes/arm_6_link.stl
- link arm_7_link: geometry collision mesh filename=/data/neobotixschunk/meshes/arm_7_link.stl scale=0.9 0.9 0.9; visual mesh filename=/data/neobotixschunk/meshes/arm_7_link.stl
- link arm_podest_link: geometry collision mesh filename=/data/neobotixschunk/meshes/arm_podest_link.stl; visual mesh filename=/data/neobotixschunk/meshes/arm_podest_link.stl
- link base_link: mass 15 -> 20; geometry collision mesh filename=/data/neobotixschunk/meshes/MP500-BODY.STL scale=0.01 0.01 0.01; visual mesh filename=/data/neobotixschunk/meshes/MP500-BODY.STL scale=0.01 0.01 0.01
- link gripper_palm_link: geometry collision box size=0.082 0.114 0.0780; visual mesh filename=/data/neobotixschunk/meshes/pg70.dae
- link gripper_podest_link: geometry collision mesh filename=/data/neobotixschunk/meshes/arm_base_link.stl; visual mesh filename=/data/neobotixschunk/meshes/arm_base_link.stl
- link hanger: geometry collision mesh filename=/data/neobotixschunk/meshes/HANGER-WHEEL.STL scale=0.01 0.01 0.01; visual mesh filename=/data/neobotixschunk/meshes/HANGER-WHEEL.STL scale=0.01 0.01 0.01
- link laserscanner_front_link: geometry collision cylinder length=0.154 radius=0.053; visual mesh filename=/data/neobotixschunk/meshes/SICK-S300.STL
- link wheel_left_link: geometry collision cylinder length=0.085 radius=0.125; visual mesh filename=/data/neobotixschunk/meshes/MP500-WHEEL.STL scale=0.01 0.01 0.01
- link wheel_right_link: geometry collision cylinder length=0.085 radius=0.125; visual mesh filename=/data/neobotixschunk/meshes/MP500-WHEEL.STL scale=0.01 0.01 0.01
Joints:
- joint arm_1_joint: origin xyz=0 0 0.019 rpy=0 0 0 -> xyz=0 0 0.02 rpy=0 0 0
- joint arm_2_joint: limit lower=-2.12 upper=2.12 effort=216 velocity=0.43633 -> lower=-2.04 upper=2.04 effort=216 velocity=0.43633
- joint arm_4_joint: limit lower=-2.16 upper=2.16 effort=81.5 velocity=0.4189 -> lower=-2.08 upper=2.08 effort=81.5 velocity=0.4189
- joint arm_6_joint: limit lower=-2.94 upper=2.94 effort=15 velocity=1.2566 -> lower=-2.08 upper=2.08 effort=15 velocity=1.2566
- joint arm_base_joint: origin xyz=0 0 0.141 rpy=0 0 0 -> xyz=0 0 0.140 rpy=0 0 0
- joint arm_podest_joint: origin xyz=0.35 0 0.36 rpy=0 0 0 -> xyz=0.19 0 0.36 rpy=0 0 0
- joint gripper_palm_joint: origin xyz=0 0 0 rpy=0 0 0 -> xyz=0 0 0.009 rpy=0 0 0
- joint hanger_joint: origin xyz=0.415 0 0.125 rpy=0 0 0 -> xyz=0.255 0 0.125 rpy=0 0 0
- joint laserscanner_front_joint: origin xyz=-0.23 0 0.281 rpy=0 0 0 -> xyz=-0.39 0 0.281 rpy=0 0 0
- joint wheel_left_joint: origin xyz=-0.01 0.255 0.125 rpy=0 0 0 -> xyz=-0.155 0.255 0.125 rpy=0 0 0
- joint wheel_right_joint: origin xyz=-0.01 -0.255 0.125 rpy=0 0 0 -> xyz=-0.155 -0.255 0.125 rpy=0 0 0
